Commit message: working joint controllers

File: src/maurice_description/urdf/macros.xacro (robot description, xacro)
@@ -1,18 +1,18 @@
 <?xml version="1.0"?>
-<robot>
-	<macro name="cylinder_inertia" params="m r h">
+<robot name="maurice" xmlns:xacro="http://www.ros.org/wiki/xacro">
+	<xacro:macro name="cylinder_inertia" params="m r h">
 		    <inertia  ixx="${m*(3*r*r+h*h)/12.0}" ixy = "0" ixz = "0"
 		                iyy="${m*(3*r*r+h*h)/12.0}" iyz = "0"
 		                izz="${m*r*r/2}" />
-		    </macro>
-	<macro name="box_inertia" params="m x y z">
+  </xacro:macro>
+	<xacro:macro name="box_inertia" params="m x y z">
 		      <inertia  ixx="${m*(y*y+z*z)/12.0}" ixy = "0" ixz = "0"
 		                iyy="${m*(x*x+z*z)/12.0}" iyz = "0"
 		                izz="${m*(x*x+z*z)/12.0}" />
-	</macro>
-	<macro name="sphere_inertia" params="m r">
+	</xacro:macro>
+	<xacro:macro name="sphere_inertia" params="m r">
 		      <inertia  ixx="${2*m*r*r/5.0}" ixy = "0" ixz = "0"
 		                iyy="${2*m*r*r/5.0}" iyz = "0"
 		                izz="${2*m*r*r/5.0}" />
-	</macro>
+	</xacro:macro>
 </robot>

File: src/maurice_description/urdf/materials.xacro (robot description, xacro)
@@ -1,4 +1,4 @@
 <?xml version="1.0" ?>
-<robot>
+<robot name="maurice" xmlns:xacro="http://www.ros.org/wiki/xacro">
   <material name="black">
     <color rgba="0.0 0.0 0.0 1.0"/>

File: src/maurice_description/urdf/maurice.xacro (robot description, xacro)
@@ -1,5 +1,5 @@
 <?xml version="1.0"?>
-<!-- Revolute-Revolute Manipulator -->
-<robot name="rrbot" xmlns:xacro="http://www.ros.org/wiki/xacro">
+<!-- Maurice Grassley-->
+<robot name="maurice" xmlns:xacro="http://www.ros.org/wiki/xacro">
   <!-- Constants for robot dimensions -->
   <xacro:property name="PI" value="3.1415926535897931"/>
@@ -311,6 +311,4 @@
       so that ros and opencv can operate on the camera frame correctly -->
   <joint name="camera_optical_joint" type="fixed">
-    <!-- these values have to be these values otherwise the gazebo camera image
-        won't be aligned properly with the frame it is supposedly originating from -->
     <origin xyz="0 0 0" rpy="${-PI/2} 0 ${-PI/2}"/>
     <parent link="camera_link"/>
