Commit message: cmd vel node

File: src/maurice_description/urdf/maurice.xacro (robot description, xacro)
@@ -226,5 +226,5 @@
     <child link="left_wheel"/>
     <origin rpy="0 0 0" xyz="0 ${wheel_track/2} -${wheel_offset}"/>
-    <axis xyz="0 -1 0"/>
+    <axis xyz="0 1 0"/>
     <dynamics damping="0.7"/>
   </joint>

Commit message: odom node

File: src/maurice_description/urdf/maurice.xacro (robot description, xacro)
@@ -198,5 +198,5 @@
     <child link="right_wheel"/>
     <origin rpy="0 0 0" xyz="0 -${wheel_track/2} -${wheel_offset}"/>
-    <axis xyz="0 -1 0"/>
+    <axis xyz="0 1 0"/>
     <dynamics damping="0.7"/>
   </joint>

Commit message: renamed robo_mower, incorporated imu and hardware package

File: src/maurice_description/urdf/maurice.xacro (robot description, xacro)
@@ -19,6 +19,8 @@
 	<xacro:property name="wheel_mass" value="1" />
 	<xacro:property name="caster_size" value="0.05" />
-  <xacro:property name="camera_link" value="0.05" />
+  <xacro:property name="camera_size" value="0.05" />
 	<xacro:property name="camera_height" value="0.1" />
+  <xacro:property name="imu_offset" value="0.15" />
+  <xacro:property name="imu_size" value="0.02" />
   <xacro:property name="axel_offset" value="0.05" /> <!-- Space btw top of beam and the each joint -->
   <!-- Import all Gazebo-customization elements, including Gazebo colors -->
@@ -281,4 +283,31 @@
     <origin rpy="0 0 0" xyz="${wheel_base} ${wheel_track/2} -${wheel_dia/2 + wheel_offset - caster_size}"/>
   </joint>
+  <!-- IMU -->
+  <link name="imu_link">
+    <collision>
+      <origin xyz="0 0 0" rpy="0 0 0"/>
+      <geometry>
+				<box size="${imu_size} ${imu_size} ${imu_size}"/>
+      </geometry>
+    </collision>
+    <visual>
+      <origin xyz="0 0 0" rpy="0 0 0"/>
+      <geometry>
+	<box size="${imu_size} ${imu_size} ${imu_size}"/>
+      </geometry>
+      <material name="blue"/>
+    </visual>
+    <inertial>
+      <mass value="1e-5" />
+      <origin xyz="0 0 0" rpy="0 0 0"/>
+      <inertia ixx="1e-6" ixy="0" ixz="0" iyy="1e-6" iyz="0" izz="1e-6" />
+    </inertial>
+  </link>
+  <joint name="base_link_to_imu_link" type="fixed">
+		<parent link="base_link"/>
+    <child link="imu_link"/>
+    <axis xyz="0 0 0" />
+    <origin xyz="-${imu_offset} 0 0" rpy="0 0 0"/>
+  </joint>
   <!-- Camera -->
   <link name="camera_link">
@@ -286,11 +315,11 @@
       <origin xyz="0 0 0" rpy="0 0 0"/>
       <geometry>
-				<box size="${camera_link} ${camera_link} ${camera_link}"/>
-      </geometry>
-    </collision>
-    <visual>
-      <origin xyz="0 0 0" rpy="0 0 0"/>
-      <geometry>
-	<box size="${camera_link} ${camera_link} ${camera_link}"/>
+				<box size="${camera_size} ${camera_size} ${camera_size}"/>
+      </geometry>
+    </collision>
+    <visual>
+      <origin xyz="0 0 0" rpy="0 0 0"/>
+      <geometry>
+	<box size="${camera_size} ${camera_size} ${camera_size}"/>
       </geometry>
       <material name="red"/>
